File: Alimentación.kicad_sch (KiCad schematic)
At the start: 1 part, among them IC1 LDO40LPURY

Commit message: .
Parts:
- IC1: footprint SON95P300X300X90-7N-D -> Transformer_SMD:Transformer_NF_ETAL_P2781_HandSoldering
Changed lines of the file:
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@@
 			)
 		)
-		(property "Footprint" "SON95P300X300X90-7N-D"
+		(property "Footprint" "Transformer_SMD:Transformer_NF_ETAL_P2781_HandSoldering"
 			(at 161.29 160.96 0)
 			(hide yes)
