File: Microcontrolador.kicad_sch (KiCad schematic)
At the start: 1 part, among them IC2 R7F125FPL4AFB-C#UA0

Commit message: .
Parts:
- IC2: footprint QFP50P1600X1600X160-100N -> Package_QFP:TQFP-100_12x12mm_P0.4mm
Changed lines of the file:
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@@
 			)
 		)
-		(property "Footprint" "QFP50P1600X1600X160-100N"
+		(property "Footprint" "Package_QFP:TQFP-100_12x12mm_P0.4mm"
 			(at 387.35 65.71 0)
-			(hide yes)
 			(show_name no)
 			(do_not_autoplace no)
